Commit message: Revert "Merge branch 'main' of https://github.com/NVlabs/curobo into devel"
This reverts commit b0cfae038d878f37259743449febf667c86a7686, reversing
changes made to 8f7b2345aef01b7980697d3ae1c09243f0eabbb7.

File: src/curobo/content/assets/robot/franka_description/franka_panda.urdf (robot description, URDF)
Before this commit: robot panda, 15 links, 14 joints
Links:
- link panda_link1: mass 2.797 -> None
- link panda_link2: mass 2.542 -> None
- link panda_link3: mass 2.2513 -> None
- link panda_link4: mass 2.2037 -> None
- link panda_link5: mass 2.2855 -> None
- link panda_link6: mass 1.353 -> None
- link panda_link7: mass 0.35973 -> None
